File: pcb/DeskHop_JLCPCB.kicad_pcb (KiCad board)
At the start: 2 copper layers, 66.9 x 74.5 mm, 12 parts, among them J1 Keyboard In, J2 Debug2, J3 Debug1, J4 Mouse In, U1 Pico Primary, U2 Pico Secondary, U4 ADuM1201BR

Commit message: Initial commit of JLCPCB-specific version.
Parts:
- J1, J4: footprint Connector_USB:USB_A_Molex_67643_Horizontal -> LCSC_C42411:USB-A-TH_JTJ-USB-10.6-002
- U4: value ADuM1201BR -> ISO7721DR
- moved J1 7.21 mm to (84.5, 107.9)
- moved J4 7.00 mm to (49.3, 107.6)
Connections:
- net /UART A TX renamed UART A TX
- net /UART B RX renamed UART B RX
- net /UART B TX renamed UART B TX
- net Net-(J1-VBUS) renamed VBUS1
- net Net-(J4-VBUS) renamed VBUS2
- net Net-(U2-3V3) renamed 3V3_BUS2
- U1 pad 17: unconnected-(U1-GPIO13-Pad17) -> UART A RX
- U4 pad 6: (no net) -> UART A RX
Routing:
- net unconnected-(U1-GPIO13-Pad17): track 6.71 -> 0.00 mm
- net UART A RX: track 0.00 -> 6.35 mm
- net Net-(J1-D-): track 11.2 -> 15.9 mm
- net Net-(J4-D-): track 13.1 -> 16.1 mm
- net VBUS2: track 94.6 -> 92.1 mm
- net VBUS1: track 91.9 -> 89.4 mm
- net Net-(J4-D+): track 15.7 -> 18.1 mm
- net Net-(J1-D+): track 15.6 -> 17.9 mm
- net Net-(J2-Pin_3): track 21.4 -> 19.6 mm
