File: pcb/DeskHop_JLCPCB.kicad_sch (KiCad schematic)
At the start: 12 parts, among them J1 Keyboard In, J2 Debug2, J3 Debug1, J4 Mouse In, U1 Pico Primary, U2 Pico Secondary, U4 ADuM1201BR

Commit message: Initial commit of JLCPCB-specific version.
Parts:
- C1, C2: LCSC (none) -> C2858367
- J1, J4: footprint Connector_USB:USB_A_Molex_67643_Horizontal -> LCSC_C42411:USB-A-TH_JTJ-USB-10.6-002; symbol Connector:USB_A -> LCSC_C42411:LCSC_C42411{colon}USB-A-TH_JTJ-USB-10.6-002; LCSC (none) -> C42411
- J2, J3: LCSC (none) -> C2915006
- U1, U2: LCSC (none) -> PICO
- U4: value ADuM1201BR -> ISO7721DR; LCSC (none) -> C366164
Connections:
- net GND: now also J4.6
- net GND2: now also J1.6
Other:
- title: DeskHop - Fast Keyboard/Mouse Switching Device -> DeskHop - Fast K/M Switching Device (JLCPCB build)
