File: pcb/core.kicad_sch (KiCad schematic)
At the start: 38 parts, among them J201 Debug, J202 Computer, J203 Power, J204 Device, Q201 USB Power Switch, U201 16Mb NOR Flash, U202 3V3 250ma LDO Regulator, U203 Microcontroller, X201 12MHz CMOS Oscillator

Commit message: Add test points for power supplies and oscillator.
Parts:
- added TP201, TP202, TP203, TP204, TP205: TestPoint_Alt, TestPoint:TestPoint_Pad_1.0x1.0mm, symbol Connector:TestPoint_Alt
Connections:
- net 3V3: now also TP204.1
- net VUSB: now also TP203.1
- net VUSB_COMP: now also TP202.1
- net VUSB_PWR: now also TP201.1
- net at U203.20 (XIN), X201.3 (OUTPUT): now also TP205.1
Other:
- moved on the sheet: R205, R206

Commit message: Update schematic with MPN/LCSC, and update manual BOM.
Parts:
- C201, C203, C204: LCSC (none) -> C541409; MPN (none) -> CC0402KRX5R5BB225
- C205, C206, C207, C208, C209, C210, C211, C212: LCSC (none) -> C541405; MPN (none) -> CC0402KRX5R5BB104
- C214, C215: LCSC (none) -> C106253; MPN (none) -> CC0402KRX5R5BB105
- D201: MPN (none) -> NCD0805B2APG1608CGKC/T
- D202: LCSC (none) -> C2828424; LCSC Part C2828424 -> (none); MPN (none) -> 1N5817WS
- J201: LCSC C2915006 -> (none)
- J202, J203, J204: MPN (none) -> GT-USB-7010ASV
- KEY201: LCSC (none) -> C86487; LCSC Part C86487 -> (none); MPN (none) -> 4-1437565-2
- Q201: LCSC (none) -> C2940629; LCSC Part C2940629 -> (none); MPN (none) -> DMG2305UX
- R201: LCSC (none) -> C144789; MPN (none) -> AC0402FR-071KL
- R202: LCSC (none) -> C227095; MPN (none) -> AC0402FR-07470RL
- R203, R204, R205, R206: LCSC (none) -> C138021; MPN (none) -> RC0402FR-0727RL
- R207, R208, R210, R211: LCSC (none) -> C144745; MPN (none) -> AC0402FR-075K1L
- R209, R212, R213: LCSC (none) -> C144778; MPN (none) -> AC0402FR-0722KL
- U201: LCSC (none) -> C82317; LCSC Part C82317 -> (none); MPN (none) -> W25Q16JVSSIQ
- U202: LCSC (none) -> C347376; LCSC Part C347376 -> (none); MPN (none) -> XC6206P332MR
- U203: LCSC (none) -> C2040; LCSC Part C2040 -> (none); MPN (none) -> RP2040
- X201: LCSC (none) -> C387348; LCSC Part C387348 -> (none); MPN (none) -> S3D12.000000B20F30T

Commit message: Add decoupling caps for oscillators.
Parts:
- added C202: 100n, Capacitor_SMD:C_0402_1005Metric, symbol Device:C
Connections:
- net 3V3: now also C202.1
- net GND: now also C202.2
Changed lines of the file:
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@@
   (junction (at 27.94 180.34) (diameter 0) (color 0 0 0 0)
+  )
+  (junction (at 58.42 90.17) (diameter 0) (color 0 0 0 0)
   )
   (junction (at 201.93 76.2) (diameter 0) (color 0 0 0 0)
@@
     (stroke (width 0) (type default))
   )
+  (wire (pts (xy 58.42 90.17) (xy 59.69 90.17))
+    (stroke (width 0) (type default))
+  )
   (wire (pts (xy 250.19 139.7) (xy 250.19 142.24))
     (stroke (width 0) (type default))
@@
     (stroke (width 0) (type default))
   )
+  (wire (pts (xy 58.42 87.63) (xy 58.42 90.17))
+    (stroke (width 0) (type default))
+  )
   (wire (pts (xy 250.19 142.24) (xy 255.27 142.24))
     (stroke (width 0) (type default))
@@
     (stroke (width 0) (type default))
   )
-  (wire (pts (xy 57.15 90.17) (xy 59.69 90.17))
+  (wire (pts (xy 57.15 90.17) (xy 58.42 90.17))
     (stroke (width 0) (type default))
   )
@@
   )
   (label "GND" (at 30.48 35.56 0) (fields_autoplaced)
+    (effects (font (size 1.27 1.27)) (justify left bottom))
+  )
+  (label "GND" (at 58.42 80.01 0) (fields_autoplaced)
     (effects (font (size 1.27 1.27)) (justify left bottom))
   )
@@
         )
       )
+    )
+  )
+  (symbol (lib_id "Device:C") (at 58.42 83.82 180) (unit 1)
+    (in_bom yes) (on_board yes) (dnp no) (fields_autoplaced)
+    (property "Reference" "C202" (at 62.23 82.55 0)
+      (effects (font (size 1.27 1.27)) (justify right))
+    )
+    (property "Value" "100n" (at 62.23 85.09 0)
+      (effects (font (size 1.27 1.27)) (justify right))
+    )
+    (property "Footprint" "Capacitor_SMD:C_0402_1005Metric" (at 57.4548 80.01 0)
+      (effects (font (size 1.27 1.27)) hide)
+    )
+    (property "Datasheet" "~" (at 58.42 83.82 0)
+      (effects (font (size 1.27 1.27)) hide)
+    )
+    (property "LCSC" "C541405" (at 58.42 83.82 0)
+      (effects (font (size 1.27 1.27)) hide)
+    )
+    (property "MPN" "CC0402KRX5R5BB104" (at 58.42 83.82 0)
+      (effects (font (size 1.27 1.27)) hide)
+    )
+    (pin "1")
+    (pin "2")
+    (instances
+      (project "DeskHop-C-JLCPCB"
+        (path "/fa1c3e0e-91b1-4532-8b22-6d396d71c75b/f9f1b756-2837-49ba-9cd6-6a0304ce3710"
+          (reference "C202") (unit 1)
+        )
+        (path "/fa1c3e0e-91b1-4532-8b22-6d396d71c75b/62cc2993-706a-4cbe-b6be-0f16bab4a3f0"
+          (reference "C302") (unit 1)
+        )
+      )

Commit message: More improvements:
* Used different GPIOs for the device USB so the traces can be kept
  away from the 12MHz oscillator circuit.

* Increased size of VBUS traces so that 1.5A@5V can be safely carried
  from the input connectors to the output connectors.

* Various minor tweaks.
Connections:
- net at R206.2: now also U203.15 (GPIO12); no longer U203.17 (GPIO14)
- net at U203.16 (GPIO13): now also R205.2
- net at U203.18 (GPIO15): no longer R205.2
Other:
- moved on the sheet: R205, R206
Changed lines of the file:
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@@
   (no_connect (at 134.62 72.39))
   (no_connect (at 250.19 92.71))
-  (no_connect (at 134.62 90.17))
+  (no_connect (at 134.62 95.25))
   (no_connect (at 134.62 62.23))
   (no_connect (at 260.35 92.71))
@@
   (no_connect (at 134.62 107.95))
   (no_connect (at 245.11 41.91))
-  (no_connect (at 134.62 87.63))
+  (no_connect (at 134.62 92.71))
   (no_connect (at 260.35 41.91))
   (no_connect (at 134.62 67.31))
@@
     (stroke (width 0) (type default))
   )
+  (wire (pts (xy 134.62 87.63) (xy 151.13 87.63))
+    (stroke (width 0) (type default))
+  )
   (wire (pts (xy 265.43 139.7) (xy 265.43 148.59))
     (stroke (width 0) (type default))
@@
     (stroke (width 0) (type default))
   )
+  (wire (pts (xy 134.62 90.17) (xy 151.13 90.17))
+    (stroke (width 0) (type default))
+  )
   (wire (pts (xy 267.97 96.52) (xy 271.78 96.52))
     (stroke (width 0) (type default))
   )
-  (wire (pts (xy 201.93 92.71) (xy 201.93 142.24))
+  (wire (pts (xy 201.93 87.63) (xy 201.93 142.24))
     (stroke (width 0) (type default))
   )
@@
     (stroke (width 0) (type default))
   )
-  (wire (pts (xy 134.62 95.25) (xy 151.13 95.25))
-    (stroke (width 0) (type default))
-  )
   (wire (pts (xy 55.88 143.51) (xy 58.42 143.51))
     (stroke (width 0) (type default))
@@
     (stroke (width 0) (type default))
   )
-  (wire (pts (xy 158.75 92.71) (xy 201.93 92.71))
-    (stroke (width 0) (type default))
-  )
-  (wire (pts (xy 134.62 92.71) (xy 151.13 92.71))
+  (wire (pts (xy 158.75 87.63) (xy 201.93 87.63))
     (stroke (width 0) (type default))
   )
@@
     (stroke (width 0) (type default))
   )
-  (wire (pts (xy 158.75 95.25) (xy 199.39 95.25))
+  (wire (pts (xy 158.75 90.17) (xy 199.39 90.17))
     (stroke (width 0) (type default))
   )
@@
     (stroke (width 0) (type default))
   )
-  (wire (pts (xy 199.39 95.25) (xy 199.39 144.78))
+  (wire (pts (xy 199.39 90.17) (xy 199.39 144.78))
     (stroke (width 0) (type default))
   )
@@
     )
   )
-  (symbol (lib_id "Device:R") (at 154.94 92.71 270) (unit 1)
+  (symbol (lib_id "Device:R") (at 154.94 87.63 270) (unit 1)
     (in_bom yes) (on_board yes) (dnp no)
-    (property "Reference" "R206" (at 154.94 97.79 90)
+    (property "Reference" "R206" (at 154.94 92.71 90)
       (effects (font (size 1.27 1.27)))
     )
-    (property "Value" "27R" (at 154.94 100.33 90)
+    (property "Value" "27R" (at 154.94 95.25 90)
       (effects (font (size 1.27 1.27)))
     )
-    (property "Footprint" "Resistor_SMD:R_0402_1005Metric" (at 154.94 90.932 90)
-      (effects (font (size 1.27 1.27)) hide)
-    )
-    (property "Datasheet" "~" (at 154.94 92.71 0)
-      (effects (font (size 1.27 1.27)) hide)
-    )
-    (property "LCSC" "C138021" (at 154.94 92.71 0)
-      (effects (font (size 1.27 1.27)) hide)
-    )
-    (property "MPN" "RC0402FR-0727RL" (at 154.94 92.71 0)
+    (property "Footprint" "Resistor_SMD:R_0402_1005Metric" (at 154.94 85.852 90)
+      (effects (font (size 1.27 1.27)) hide)
+    )
+    (property "Datasheet" "~" (at 154.94 87.63 0)
+      (effects (font (size 1.27 1.27)) hide)
+    )
+    (property "LCSC" "C138021" (at 154.94 87.63 0)
+      (effects (font (size 1.27 1.27)) hide)
+    )
+    (property "MPN" "RC0402FR-0727RL" (at 154.94 87.63 0)
       (effects (font (size 1.27 1.27)) hide)
     )
@@
     )
   )
-  (symbol (lib_id "Device:R") (at 154.94 95.25 270) (unit 1)
+  (symbol (lib_id "Device:R") (at 154.94 90.17 270) (unit 1)
     (in_bom yes) (on_board yes) (dnp no)
-    (property "Reference" "R205" (at 154.94 87.63 90)
+    (property "Reference" "R205" (at 154.94 82.55 90)
       (effects (font (size 1.27 1.27)))
     )
-    (property "Value" "27R" (at 154.94 90.17 90)
+    (property "Value" "27R" (at 154.94 85.09 90)
       (effects (font (size 1.27 1.27)))
     )
-    (property "Footprint" "Resistor_SMD:R_0402_1005Metric" (at 154.94 93.472 90)
-      (effects (font (size 1.27 1.27)) hide)
-    )
-    (property "Datasheet" "~" (at 154.94 95.25 0)
-      (effects (font (size 1.27 1.27)) hide)
-    )
-    (property "LCSC" "C138021" (at 154.94 95.25 0)
-      (effects (font (size 1.27 1.27)) hide)
-    )
-    (property "MPN" "RC0402FR-0727RL" (at 154.94 95.25 0)
-      (effects (font (size 1.27 1.27)) hide)
-    )
+    (property "Footprint" "Resistor_SMD:R_0402_1005Metric" (at 154.94 88.392 90)
+      (effects (font (size 1.27 1.27)) hide)
+    )
+    (property "Datasheet" "~" (at 154.94 90.17 0)
+      (effects (font (size 1.27 1.27)) hide)
+    )
+    (property "LCSC" "C138021" (at 154.94 90.17 0)
+      (effects (font (size 1.27 1.27)) hide)
+    )
+    (property "MPN" "RC0402FR-0727RL" (at 154.94 90.17 0)
+      (effects (font (size 1.27 1.27)) hide)
+    )

Commit message: Use better net labels for UART links.
Connections:
- net UART-RX-A renamed RIGHT-UART-RX
- net UART-RX-B renamed LEFT-UART-RX
- net UART-TX-A renamed RIGHT-UART-TX
- net UART-TX-B renamed LEFT-UART-TX
Other:
- moved on the sheet: R205, R206
Changed lines of the file:
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@@
     (stroke (width 0) (type default))
   )
-  (wire (pts (xy 134.62 87.63) (xy 151.13 87.63))
+  (wire (pts (xy 134.62 87.63) (xy 158.75 87.63))
     (stroke (width 0) (type default))
   )
@@
     (stroke (width 0) (type default))
   )
-  (wire (pts (xy 134.62 90.17) (xy 151.13 90.17))
+  (wire (pts (xy 134.62 90.17) (xy 158.75 90.17))
     (stroke (width 0) (type default))
   )
@@
     (stroke (width 0) (type default))
   )
-  (wire (pts (xy 158.75 87.63) (xy 201.93 87.63))
+  (wire (pts (xy 166.37 87.63) (xy 201.93 87.63))
     (stroke (width 0) (type default))
   )
@@
     (stroke (width 0) (type default))
   )
-  (wire (pts (xy 158.75 90.17) (xy 199.39 90.17))
+  (wire (pts (xy 166.37 90.17) (xy 199.39 90.17))
     (stroke (width 0) (type default))
   )
@@
     (effects (font (size 1.27 1.27)) (justify left bottom))
   )
-  (hierarchical_label "UART-RX-A" (shape input) (at 138.43 85.09 0) (fields_autoplaced)
+  (hierarchical_label "RIGHT-UART-RX" (shape input) (at 138.43 85.09 0) (fields_autoplaced)
     (effects (font (size 1.27 1.27)) (justify left))
   )
@@
     (effects (font (size 1.27 1.27)) (justify left))
   )
-  (hierarchical_label "UART-RX-B" (shape input) (at 138.43 105.41 0) (fields_autoplaced)
+  (hierarchical_label "LEFT-UART-RX" (shape input) (at 138.43 105.41 0) (fields_autoplaced)
     (effects (font (size 1.27 1.27)) (justify left))
   )
-  (hierarchical_label "UART-TX-A" (shape output) (at 138.43 82.55 0) (fields_autoplaced)
+  (hierarchical_label "RIGHT-UART-TX" (shape output) (at 138.43 82.55 0) (fields_autoplaced)
     (effects (font (size 1.27 1.27)) (justify left))
   )
@@
     (effects (font (size 1.27 1.27)) (justify left))
   )
-  (hierarchical_label "UART-TX-B" (shape output) (at 138.43 102.87 0) (fields_autoplaced)
+  (hierarchical_label "LEFT-UART-TX" (shape output) (at 138.43 102.87 0) (fields_autoplaced)
     (effects (font (size 1.27 1.27)) (justify left))
   )
@@
     )
   )
-  (symbol (lib_id "Device:R") (at 154.94 87.63 270) (unit 1)
+  (symbol (lib_id "Device:R") (at 162.56 87.63 270) (unit 1)
     (in_bom yes) (on_board yes) (dnp no)
-    (property "Reference" "R206" (at 154.94 92.71 90)
+    (property "Reference" "R206" (at 162.56 92.71 90)
       (effects (font (size 1.27 1.27)))
     )
-    (property "Value" "27R" (at 154.94 95.25 90)
+    (property "Value" "27R" (at 162.56 95.25 90)
       (effects (font (size 1.27 1.27)))
     )
-    (property "Footprint" "Resistor_SMD:R_0402_1005Metric" (at 154.94 85.852 90)
-      (effects (font (size 1.27 1.27)) hide)
-    )
-    (property "Datasheet" "~" (at 154.94 87.63 0)
-      (effects (font (size 1.27 1.27)) hide)
-    )
-    (property "LCSC" "C138021" (at 154.94 87.63 0)
-      (effects (font (size 1.27 1.27)) hide)
-    )
-    (property "MPN" "RC0402FR-0727RL" (at 154.94 87.63 0)
+    (property "Footprint" "Resistor_SMD:R_0402_1005Metric" (at 162.56 85.852 90)
+      (effects (font (size 1.27 1.27)) hide)
+    )
+    (property "Datasheet" "~" (at 162.56 87.63 0)
+      (effects (font (size 1.27 1.27)) hide)
+    )
+    (property "LCSC" "C138021" (at 162.56 87.63 0)
+      (effects (font (size 1.27 1.27)) hide)
+    )
+    (property "MPN" "RC0402FR-0727RL" (at 162.56 87.63 0)
       (effects (font (size 1.27 1.27)) hide)
     )
@@
     )
   )
-  (symbol (lib_id "Device:R") (at 154.94 90.17 270) (unit 1)
+  (symbol (lib_id "Device:R") (at 162.56 90.17 270) (unit 1)
     (in_bom yes) (on_board yes) (dnp no)
-    (property "Reference" "R205" (at 154.94 82.55 90)
+    (property "Reference" "R205" (at 162.56 82.55 90)
       (effects (font (size 1.27 1.27)))
     )
-    (property "Value" "27R" (at 154.94 85.09 90)
+    (property "Value" "27R" (at 162.56 85.09 90)
       (effects (font (size 1.27 1.27)))
     )
-    (property "Footprint" "Resistor_SMD:R_0402_1005Metric" (at 154.94 88.392 90)
-      (effects (font (size 1.27 1.27)) hide)
-    )
-    (property "Datasheet" "~" (at 154.94 90.17 0)
-      (effects (font (size 1.27 1.27)) hide)
-    )
-    (property "LCSC" "C138021" (at 154.94 90.17 0)
-      (effects (font (size 1.27 1.27)) hide)
-    )
-    (property "MPN" "RC0402FR-0727RL" (at 154.94 90.17 0)
-      (effects (font (size 1.27 1.27)) hide)
-    )
+    (property "Footprint" "Resistor_SMD:R_0402_1005Metric" (at 162.56 88.392 90)
+      (effects (font (size 1.27 1.27)) hide)
+    )
+    (property "Datasheet" "~" (at 162.56 90.17 0)
+      (effects (font (size 1.27 1.27)) hide)
+    )
+    (property "LCSC" "C138021" (at 162.56 90.17 0)
+      (effects (font (size 1.27 1.27)) hide)
+    )
+    (property "MPN" "RC0402FR-0727RL" (at 162.56 90.17 0)
+      (effects (font (size 1.27 1.27)) hide)
+    )

Commit message: Lots of improvements:
* Modified footprint for USB Type-C connector to use an NPTH for the
  plastic locator pins.

* Connected USB SHIELD to GND as required by the USB spec.

* Simplified trace routing and eliminated most vias.

* Improved VUSB trace routing and sizing.
Connections:
- net SHIELD is gone; now on net GND: J202.1 (SHELL), J202.2 (SHELL), J202.3 (SHELL), J202.4 (SHELL), J203.1 (SHELL), J203.2 (SHELL), J203.3 (SHELL), J203.4 (SHELL), J204.1 (SHELL), J204.2 (SHELL), J204.3 (SHELL), J204.4 (SHELL)
Changed lines of the file:
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@@
   (title_block
     (title "DeskHop-C - Fast K/M Switching Device (JLCPCB build)")
-    (date "2024-03-17")
+    (date "2024-03-22")
     (rev "v1-jlcpcb")
     (company "Hrvoje Čavrak and Kevin P. Fleming")
@@
   (junction (at 187.96 44.45) (diameter 0) (color 0 0 0 0)
   )
-  (junction (at 46.99 58.42) (diameter 0) (color 0 0 0 0)
-  )
   (junction (at 265.43 69.85) (diameter 0) (color 0 0 0 0)
   )
@@
   (junction (at 242.57 19.05) (diameter 0) (color 0 0 0 0)
   )
+  (junction (at 26.67 58.42) (diameter 0) (color 0 0 0 0)
+  )
   (junction (at 265.43 50.8) (diameter 0) (color 0 0 0 0)
   )
@@
   (junction (at 93.98 38.1) (diameter 0) (color 0 0 0 0)
   )
+  (junction (at 41.91 58.42) (diameter 0) (color 0 0 0 0)
+  )
   (junction (at 33.02 182.88) (diameter 0) (color 0 0 0 0)
   )
@@
   )
   (junction (at 250.19 142.24) (diameter 0) (color 0 0 0 0)
-  )
-  (junction (at 21.59 58.42) (diameter 0) (color 0 0 0 0)
   )
   (junction (at 262.89 110.49) (diameter 0) (color 0 0 0 0)
@@
     (stroke (width 0) (type default))
   )
-  (wire (pts (xy 41.91 58.42) (xy 46.99 58.42))
+  (wire (pts (xy 41.91 58.42) (xy 52.07 58.42))
     (stroke (width 0) (type default))
   )
@@
     (stroke (width 0) (type default))
   )
-  (wire (pts (xy 21.59 58.42) (xy 26.67 58.42))
+  (wire (pts (xy 13.97 58.42) (xy 26.67 58.42))
     (stroke (width 0) (type default))
   )
@@
     (stroke (width 0) (type default))
   )
-  (wire (pts (xy 21.59 55.88) (xy 21.59 58.42))
-    (stroke (width 0) (type default))
-  )
   (wire (pts (xy 144.78 17.78) (xy 144.78 25.4))
     (stroke (width 0) (type default))
@@
     (stroke (width 0) (type default))
   )
-  (wire (pts (xy 13.97 58.42) (xy 21.59 58.42))
-    (stroke (width 0) (type default))
-  )
   (wire (pts (xy 102.87 144.78) (xy 102.87 152.4))
     (stroke (width 0) (type default))
@@
     (stroke (width 0) (type default))
   )
-  (wire (pts (xy 26.67 55.88) (xy 21.59 55.88))
-    (stroke (width 0) (type default))
-  )
   (wire (pts (xy 247.65 92.71) (xy 247.65 100.33))
     (stroke (width 0) (type default))
@@
     (stroke (width 0) (type default))
   )
-  (wire (pts (xy 46.99 58.42) (xy 52.07 58.42))
-    (stroke (width 0) (type default))
-  )
   (wire (pts (xy 265.43 69.85) (xy 267.97 69.85))
     (stroke (width 0) (type default))
@@
     (stroke (width 0) (type default))
   )
+  (wire (pts (xy 26.67 55.88) (xy 26.67 58.42))
+    (stroke (width 0) (type default))
+  )
   (wire (pts (xy 55.88 140.97) (xy 58.42 140.97))
     (stroke (width 0) (type default))
@@
     (stroke (width 0) (type default))
   )
-  (wire (pts (xy 46.99 55.88) (xy 46.99 58.42))
-    (stroke (width 0) (type default))
-  )
   (wire (pts (xy 57.15 90.17) (xy 58.42 90.17))
     (stroke (width 0) (type default))
@@
     (stroke (width 0) (type default))
   )
+  (wire (pts (xy 41.91 55.88) (xy 41.91 58.42))
+    (stroke (width 0) (type default))
+  )
   (wire (pts (xy 43.18 17.78) (xy 43.18 25.4))
     (stroke (width 0) (type default))
@@
     (stroke (width 0) (type default))
   )
-  (wire (pts (xy 41.91 55.88) (xy 46.99 55.88))
-    (stroke (width 0) (type default))
-  )
   (wire (pts (xy 242.57 69.85) (xy 265.43 69.85))
     (stroke (width 0) (type default))
@@
     (effects (font (size 1.27 1.27)) (justify left bottom))
   )
-  (label "SHIELD" (at 271.78 69.85 0) (fields_autoplaced)
-    (effects (font (size 1.27 1.27)) (justify left bottom))
-  )
-  (label "SHIELD" (at 271.78 116.84 0) (fields_autoplaced)
+  (label "GND" (at 271.78 69.85 0) (fields_autoplaced)
+    (effects (font (size 1.27 1.27)) (justify left bottom))
+  )
+  (label "GND" (at 271.78 116.84 0) (fields_autoplaced)
     (effects (font (size 1.27 1.27)) (justify left bottom))
   )
@@
     (effects (font (size 1.27 1.27)) (justify left bottom))
   )
-  (label "SHIELD" (at 271.78 19.05 0) (fields_autoplaced)
-    (effects (font (size 1.27 1.27)) (justify left bottom))
-  )
+  (label "GND" (at 271.78 19.05 0) (fields_autoplaced)
+    (effects (font (size 1.27 1.27)) (justify left bottom))
+  )
